Commit message: import Victor gripper in sim (the tool signal output doesn't align??)

File: data/grasp_screw_tool_description/urdf/grasp_screw_tool_unactuated.urdf (robot description, URDF)
Before this commit: robot grasp_screw_tool_unactuated, 2 links, 1 joints
Links:
- link grasp_screw_tool_link: geometry collision mesh filename=package://grasp_screw_tool_description/meshes/collision/gra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; visual mesh filename=package://grasp_screw_tool_description/meshes/visual/grasp_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

Commit message: change urdf of tool - visual causing GUI problem

File: data/grasp_screw_tool_description/urdf/grasp_screw_tool_unactuated.urdf (robot description, URDF)
Before this commit: robot grasp_screw_tool_unactuated, 2 links, 1 joints
Links:
- link grasp_screw_tool_link: geometry collision mesh filename=package://grasp_screw_tool_description/meshes/collision/gra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; visual mesh filename=package://grasp_screw_tool_description/meshes/collision/gra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
